File: Vent.kicad_pcb (KiCad board)
At the start: 2 copper layers, 25.5 x 60 mm, 4 parts, among them U1 ESP32-S3-WROOM-1, U2 MCP9808T-E_MS

Commit message: Autoprogramming Circuit
Original-author: Zachariah K. Sharma <zachariah.sharma@gmail.com>
Source-commit: 72ef880672316db68a35278d5394047a9c77ba1c
Parts:
- added C1: 100nF, PCM_JLCPCB:C_0805, F.Cu at (126.6, 88.0)
- added C2: 4.7uF, PCM_JLCPCB:C_0805, F.Cu at (126.6, 91.1)
- added Q1: S8050 J3Y 200-350, PCM_JLCPCB:Q_SOT-23, F.Cu at (131.3, 88.9)
- added R3: 5.1kΩ, PCM_JLCPCB:R_0603, F.Cu at (130.7, 92.2)
- added R4: 5.1kΩ, PCM_JLCPCB:R_0603, F.Cu at (130.7, 94.5)
Connections:
- U1 pad 27: unconnected-(U1-IO0-Pad27) -> IO0
- U1 pad 3: unconnected-(U1-EN-Pad3) -> EN
- U1 pad 36: unconnected-(U1-RXD0-Pad36) -> RXD0
- U1 pad 37: unconnected-(U1-TXD0-Pad37) -> TXD0

Commit message: Fixed most of the bugs hopefully
Original-author: Zachariah K. Sharma <zachariah.sharma@gmail.com>
Source-commit: 95630e4fc29616ac93e070c71f119a40b19bcd80
Parts:
- added C3: 10uF, PCM_JLCPCB:C_0603, F.Cu at (135.4, 93.8)
- added C4: 10uF, PCM_JLCPCB:C_0603, F.Cu at (135.4, 96.0)
- added C5: 1uF, PCM_JLCPCB:C_0603, F.Cu at (135.4, 98.2)
- added C6: 100nF, PCM_JLCPCB:C_0805, F.Cu at (140.6, 89.5)
- added J1: TYPE-C-31-M-12, Footprints:HRO_TYPE-C-31-M-12, F.Cu at (161.9, 76.9)
- added Q2: S8050 J3Y 200-350, PCM_JLCPCB:Q_SOT-23, F.Cu at (150.6, 90.5)
- added R5: 10kΩ, PCM_JLCPCB:R_0603, F.Cu at (139.2, 93.8)
- added R6: 10kΩ, PCM_JLCPCB:R_0603, F.Cu at (139.2, 96.0)
- added R7: 10kΩ, PCM_JLCPCB:R_0603, F.Cu at (139.2, 98.2)
- added R8: 10kΩ, PCM_JLCPCB:R_0603, F.Cu at (139.2, 100.5)
- added U3: CP2102N-A02-GQFN28R, Footprints:IC_CP2102N-A02-GQFN28R, F.Cu at (160.0, 83.9)
- added U4: AP2112K-3.3TRG1, Footprints:SOT95P285X140-5N, F.Cu at (166.8, 82.5)
- moved U1 15.2 mm to (143.8, 73.8)
- moved C2 13.0 mm to (116.5, 83.0)
- moved U2 12.8 mm to (121.5, 98.0), turned to 0 degrees
- moved Q1 11.9 mm to (119.4, 89.5)
- moved C1 10.0 mm to (127.0, 78.0)
Connections:
- Q1 pad 1: unconnected-(Q1-B-Pad1) -> Net-(Q1-B)
- Q1 pad 2: unconnected-(Q1-E-Pad2) -> GND
- Q1 pad 3: unconnected-(Q1-C-Pad3) -> EN
- U1 pad 13: unconnected-(U1-USB_D--Pad13) -> USB_D-
- U1 pad 14: unconnected-(U1-USB_D+-Pad14) -> USB_D+
- U2 pad 5: unconnected-(U2-A2-Pad5) -> GND
- U2 pad 6: unconnected-(U2-A1-Pad6) -> GND
- U2 pad 7: unconnected-(U2-A0-Pad7) -> GND
Other:
- board outline removed
