File: Temp Sensor.kicad_sch (KiCad schematic)
At the start: 3 parts, among them U5 MCP9808T-E_MS

Commit message: feat: Add metadata for schematic sheets
Original-author: Ishan Karmakar <ishan.karmakar24@gmail.com>
Source-commit: c82f4670f2f6b6f19a8645b0d3909227ee38d77d
Other:
- company: (none) -> Vynte
- title: (none) -> Temperature Sensor
Changed lines of the file:
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@@
 	(generator_version "10.0")
 	(paper "A4")
+	(title_block
+		(title "Temperature Sensor")
+		(date "2026-08-21")
+		(rev "${PROJECT_REV}")
+		(company "Vynte")
+	)
 	(junction
 		(at 107.95 99.06)
