File: ExternalAutoprogramming.kicad_sch (KiCad schematic)
At the start: 1 part, among them J4 Conn_01x04_Socket

Commit message: feat: Add metadata for schematic sheets
Original-author: Ishan Karmakar <ishan.karmakar24@gmail.com>
Source-commit: c82f4670f2f6b6f19a8645b0d3909227ee38d77d
Other:
- company: (none) -> Vynte
- title: (none) -> External Autoprogramming
Changed lines of the file:
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@@
 	(generator_version "10.0")
 	(paper "A4")
+	(title_block
+		(title "External Autoprogramming")
+		(date "2026-08-21")
+		(rev "${PROJECT_REV}")
+		(company "Vynte")
+	)
 	(wire
 		(pts

Commit message: feat: Disconnect RX and TX pins
Original-author: Ishan Karmakar <ishan.karmakar24@gmail.com>
Source-commit: 296c2ee0a068d96963a51e7bc8ff53979a0f6f0b
Connections:
- net RX: no longer names the net of J4.1 (RX)
- net TX: no longer names the net of J4.3 (TX)
- no-connect marks 0 -> 2
Changed lines of the file:
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@@
 		(company "Vynte")
+	)
+	(no_connect
+		(at 156.21 97.79)
+	)
+	(no_connect
+		(at 156.21 95.25)
 	)
 	(wire
@@
 		)
 	)
-	(hierarchical_label "TX"
-		(shape bidirectional)
-		(at 156.21 97.79 180)
-		(effects
-			(font
-				(size 1.27 1.27)
-			)
-			(justify right)
-		)
-	)
-	(hierarchical_label "RX"
-		(shape bidirectional)
-		(at 156.21 95.25 180)
-		(effects
-			(font
-				(size 1.27 1.27)
-			)
-			(justify right)
-		)
-	)

Commit message: feat: Remove the BOOT pin + NC GPIO9
Original-author: Ishan Karmakar <ishan.karmakar24@gmail.com>
Source-commit: 8bb5acb199ee9e43bb7b500971a5340ad49e3dfa
Connections:
- net BOOT: no longer names the net of J4.4 (BOOT)
- no-connect marks 2 -> 3
Changed lines of the file:
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@@
+	)
+	(no_connect
+		(at 175.26 97.79)
 	)
 	(no_connect
@@
 		)
 	)
-	(hierarchical_label "BOOT"
-		(shape bidirectional)
-		(at 175.26 97.79 0)
-		(effects
-			(font
-				(size 1.27 1.27)
-			)
-			(justify left)
-		)
-	)
