File: Type C Recepticle.kicad_sch (KiCad schematic)
At the start: 3 parts, among them J3 TYPE-C-31-M-12

Commit message: feat: Add metadata for schematic sheets
Original-author: Ishan Karmakar <ishan.karmakar24@gmail.com>
Source-commit: c82f4670f2f6b6f19a8645b0d3909227ee38d77d
Other:
- company: (none) -> Vynte
- title: (none) -> Type C Recepticle
Changed lines of the file:
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@@
 	(generator_version "10.0")
 	(paper "A4")
+	(title_block
+		(title "Type C Recepticle")
+		(date "2026-08-21")
+		(rev "${PROJECT_REV}")
+		(company "Vynte")
+	)
 	(junction
 		(at 161.29 111.76)

Commit message: feat: Wire D+ and D- from Type C recepticle to ESP32 pins
Original-author: Ishan Karmakar <ishan.karmakar24@gmail.com>
Source-commit: f485fb4ecb58e7db9c11b8a83e3a2328aeb9ad39
Connections:
- net D+: now reaches J3.A6 (DP1)
- net D+: now also J3.B6 (DP2)
- net D-: now reaches J3.A7 (DN1)
- net D-: now also J3.B7 (DN2)
- no-connect marks 6 -> 2
Changed lines of the file:
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@@
-	)
-	(no_connect
-		(at 158.75 99.06)
-	)
-	(no_connect
-		(at 123.19 101.6)
-	)
-	(no_connect
-		(at 158.75 101.6)
-	)
-	(no_connect
-		(at 123.19 99.06)
 	)
 	(no_connect
@@
 		)
 	)
+	(hierarchical_label "D-"
+		(shape input)
+		(at 158.75 99.06 0)
+		(effects
+			(font
+				(size 1.27 1.27)
+			)
+			(justify left)
+		)
+	)
+	(hierarchical_label "D-"
+		(shape input)
+		(at 123.19 101.6 180)
+		(effects
+			(font
+				(size 1.27 1.27)
+			)
+			(justify right)
+		)
+	)
+	(hierarchical_label "D+"
+		(shape input)
+		(at 123.19 99.06 180)
+		(effects
+			(font
+				(size 1.27 1.27)
+			)
+			(justify right)
+		)
+	)
+	(hierarchical_label "D+"
+		(shape input)
+		(at 158.75 101.6 0)
+		(effects
+			(font
+				(size 1.27 1.27)
+			)
+			(justify left)
+		)
+	)
