File: Puck.kicad_pcb (KiCad board)
At the start: 2 copper layers, 26.6 x 72.5 mm, 19 parts, among them J3 TYPE-C-31-M-12, J4 Conn_01x04_Socket, SW1 SW_Push, SW2 SW_Push, U1 ET6226M, U2 ESP32-C6-MINI-1/U, U4 AP2112K-3.3TRG1, U5 MCP9808T-E_MS

Commit message: feat: Use standard KiCad capacitor symbols and footprints
Original-author: Ishan Karmakar <ishan.karmakar24@gmail.com>
Source-commit: 6d92738db7c1a3a0126f93a2d140869e5f4c1fb9
Parts:
- C1: value 1 uF -> 1uF; footprint PCM_JLCPCB:C_0603 -> Capacitor_SMD:C_0603_1608Metric
- C3, C4, C5: footprint PCM_JLCPCB:C_0603 -> Capacitor_SMD:C_0603_1608Metric
- C6: footprint PCM_JLCPCB:C_0805 -> Capacitor_SMD:C_0603_1608Metric
- moved C3 0.40 mm to (155.1, 122.4)
- moved C4 0.29 mm to (155.1, 128.2)
- moved C1 0.09 mm to (159.9, 101.9)
