File: SevenSegmentDisplay.kicad_sch (KiCad schematic)
At the start: 3 parts, among them U1 ET6226M

Commit message: feat: Add metadata for schematic sheets
Original-author: Ishan Karmakar <ishan.karmakar24@gmail.com>
Source-commit: c82f4670f2f6b6f19a8645b0d3909227ee38d77d
Other:
- company: (none) -> Vynte
- title: (none) -> Seven Segment Display
Changed lines of the file:
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@@
 	(generator_version "10.0")
 	(paper "A4")
+	(title_block
+		(title "Seven Segment Display")
+		(date "2026-08-21")
+		(rev "${PROJECT_REV}")
+		(company "Vynte")
+	)
 	(junction
 		(at 201.93 77.47)

Commit message: feat: Use standard KiCad capacitor symbols and footprints
Original-author: Ishan Karmakar <ishan.karmakar24@gmail.com>
Source-commit: 6d92738db7c1a3a0126f93a2d140869e5f4c1fb9
Parts:
- removed C1: 1 uF, PCM_JLCPCB:C_0603, symbol Device:C
- added C1: 1uF, Capacitor_SMD:C_0603_1608Metric, symbol Device:C_Small
Connections:
- net +5V: now also C1.1
- net GND: now also C1.2
Changed lines of the file:
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@@
-		)
-	)
-	(wire
-		(pts
-			(xy 201.93 85.09) (xy 201.93 88.9)
-		)
-		(stroke
-			(width 0)
-			(type default)
 		)
 	)
@@
 	(symbol
 		(lib_id "power:GND")
-		(at 201.93 88.9 0)
+		(at 201.93 82.55 0)
 		(unit 1)
 		(body_style 1)
@@
 		(fields_autoplaced yes)
 		(property "Reference" "#PWR017"
-			(at 201.93 95.25 0)
+			(at 201.93 88.9 0)
 			(hide yes)
 			(show_name no)
@@
 		)
 		(property "Value" "GND"
-			(at 201.93 93.98 0)
+			(at 201.93 87.63 0)
 			(show_name no)
 			(do_not_autoplace no)
@@
 		)
 		(property "Footprint" ""
-			(at 201.93 88.9 0)
+			(at 201.93 82.55 0)
 			(hide yes)
 			(show_name no)
@@
 		)
 		(property "Datasheet" ""
-			(at 201.93 88.9 0)
+			(at 201.93 82.55 0)
 			(hide yes)
 			(show_name no)
@@
 		)
 		(property "Description" "Power symbol creates a global label with name \"GND\" , ground"
-			(at 201.93 88.9 0)
+			(at 201.93 82.55 0)
 			(hide yes)
 			(show_name no)
@@
 	)
 	(symbol
-		(lib_id "Device:C")
-		(at 201.93 81.28 0)
+		(lib_id "Device:C_Small")
+		(at 201.93 80.01 0)
 		(unit 1)
 		(body_style 1)
@@
 		(fields_autoplaced yes)
 		(property "Reference" "C1"
-			(at 205.74 80.0099 0)
+			(at 204.47 78.7462 0)
 			(show_name no)
 			(do_not_autoplace no)
@@
 			)
 		)
-		(property "Value" "1 uF"
-			(at 205.74 82.5499 0)
+		(property "Value" "1uF"
+			(at 204.47 81.2862 0)
 			(show_name no)
 			(do_not_autoplace no)
@@
 			)
 		)
-		(property "Footprint" "PCM_JLCPCB:C_0603"
-			(at 202.8952 85.09 0)
+		(property "Footprint" "Capacitor_SMD:C_0603_1608Metric"
+			(at 201.93 80.01 0)
 			(hide yes)
 			(show_name no)
@@
 		)
 		(property "Datasheet" ""
-			(at 201.93 81.28 0)
-			(hide yes)
-			(show_name no)
-			(do_not_autoplace no)
-			(effects
-				(font
-					(size 1.27 1.27)
-				)
-			)
-		)
-		(property "Description" "Unpolarized capacitor"
-			(at 201.93 81.28 0)
-			(hide yes)
-			(show_name no)
-			(do_not_autoplace no)
-			(effects
-				(font
-					(size 1.27 1.27)
-				)
-			)
-		)
-		(property "MPN" "CL10A105KB8NNNC"
-			(at 205.74 82.5499 0)
-			(hide yes)
-			(show_name no)
-			(do_not_autoplace no)
-			(effects
-				(font
-					(size 1.27 1.27)
-				)
-			)
-		)
-		(property "Manufacturer" "Samsung Electro-Mechanics"
-			(at 205.74 82.5499 0)
-			(hide yes)
-			(show_name no)
-			(do_not_autoplace no)
-			(effects
-				(font
-					(size 1.27 1.27)
-				)
-			)
-		)
-		(property "LCSC" "C15849"
-			(at 205.74 82.5499 0)
-			(hide yes)
-			(show_name no)
-			(do_not_autoplace no)
-			(effects
-				(font
-					(size 1.27 1.27)
-				)
-			)
+			(at 201.93 80.01 0)
+			(hide yes)
+			(show_name no)
+			(do_not_autoplace no)
+			(effects
+				(font
+					(size 1.27 1.27)
+				)
+			)
+		)
+		(property "Description" "Unpolarized capacitor, small symbol"
+			(at 201.93 80.01 0)
+			(hide yes)
+			(show_name no)
+			(do_not_autoplace no)
+			(effects
+				(font
+					(size 1.27 1.27)
+				)
+			)
+		)
+		(pin "1"
 		)
 		(pin "2"
 		)
-		(pin "1"
-		)
 		(instances
