File: SevenSegmentDisplay.kicad_sch (KiCad schematic)
At the start: 3 parts, among them U1 ET6226M

Commit message: feat: Preserve saved puck design and fabrication package
Original-author: Zachariah K. Sharma <zachariah.sharma@gmail.com>
Source-commit: e899556739295891c68fe5bb4e4d2c3c5016f347
Connections:
- net +5V renamed +3.3V
Changed lines of the file:
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@@
 	)
 	(symbol
-		(lib_id "power:+5V")
+		(lib_id "power:+3.3V")
 		(at 201.93 69.85 0)
 		(unit 1)
@@
 			)
 		)
-		(property "Value" "+5V"
+		(property "Value" "+3.3V"
 			(at 201.93 64.77 0)
 			(show_name no)
@@
 			)
 		)
-		(property "Description" "Power symbol creates a global label with name \"+5V\""
+		(property "Description" "Power symbol creates a global label with name \"+3.3V\""
 			(at 201.93 69.85 0)
 			(hide yes)
