File: Puck.kicad_sch (KiCad schematic)
At the start: 5 parts, among them SW1 SW_Push, SW2 SW_Push, U3 ESP32-C6-MINI-1

Commit message: feat: Preserve saved puck design and fabrication package
Original-author: Zachariah K. Sharma <zachariah.sharma@gmail.com>
Source-commit: e899556739295891c68fe5bb4e4d2c3c5016f347
Parts:
- added C3: 4.7uF, PCM_JLCPCB:C_0603, symbol Device:C
- added C7: .1uF, PCM_JLCPCB:C_0603, symbol Device:C
- SW1, SW2: footprint Footprints:SW_TS-1187A-B-A-B_2term -> Button_Switch_THT:SW_PUSH_6mm_H7.3mm; DigiKey (none) -> SW414-ND; LCSC C318884 -> (none); MPN TS-1187A-B-A-B -> B3F-4055; Manufacturer XKB Connection -> Omron Electronics
Connections:
- net +3.3V: now also C3.1, C7.1
- net GND: now also C3.2, C7.2
- no-connect marks 12 -> 13
