File: Puck/Vent.kicad_sch (KiCad schematic)
At the start: 21 parts, among them J1 TYPE-C-31-M-12, Q1 S8050 J3Y 200-350, Q2 S8050 J3Y 200-350, U1 ESP32-S3-WROOM-1, U2 MCP9808T-E_MS, U3 CP2102N-A02-GQFN28R, U4 AP2112K-3.3TRG1

Commit message: Reorganized Files
Original-author: Zachariah K. Sharma <zachariah.sharma@gmail.com>
Source-commit: 0b0902855738d5cdca35fa15d060f71b343d7e14
Other:
- note added: "PSRAM"
Changed lines of the file:
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@@
 	(text "Temperature Sensor"
 		(exclude_from_sim no)
-		(at 340.106 24.384 0)
+		(at 328.422 19.05 0)
+		(effects
+			(font
+				(size 2.54 2.54)
+			)
+		)
+	)
+	(text "PSRAM\n"
+		(exclude_from_sim no)
+		(at 316.738 173.736 0)
 		(effects
 			(font
@@
 	(text "ESP-32"
 		(exclude_from_sim no)
-		(at 333.248 87.122 0)
+		(at 318.77 87.884 0)
 		(effects
 			(font
@@
 	)
 	(junction
+		(at 304.8 167.64)
+		(diameter 0)
+		(color 0 0 0 0)
+	)
+	(junction
 		(at 66.04 236.22)
 		(diameter 0)
@@
 		)
 	)
+	(bus
+		(pts
+			(xy 304.8 234.95) (xy 419.1 234.95)
+		)
+		(stroke
+			(width 0)
+			(type default)
+		)
+	)
 	(wire
 		(pts
@@
 		)
 		(stroke
+			(width 0)
+			(type default)
+		)
+	)
+	(bus
+		(pts
+			(xy 304.8 167.64) (xy 304.8 234.95)
+		)
+		(stroke
