File: Vent/Vent.kicad_sch (KiCad schematic)
At the start: 0 parts

Commit message: Added symbols, models, footprints for BMS and added wiring for Safety and the Brain
Original-author: Zachariah K. Sharma <zachariah.sharma@gmail.com>
Source-commit: 61d43b963560d7d84e99585d61830151d00a31d1
Parts:
- added U1: ESP32-C3-WROOM-02-N4, ESP32-C3-WROOM-02-N4:MODULE_ESP32-C3-WROOM-02-H4, symbol ESP32-C3-WROOM-02-N4:ESP32-C3-WROOM-02-N4
Connections:
- new net +3V3: U1.1 (3V3)
- new net GND: U1.19 (GND), U1.20 (GND), U1.21 (GND), U1.22 (GND), U1.23 (GND), U1.24 (GND), U1.25 (GND), U1.26 (GND), U1.27 (GND), U1.28 (GND), U1.29 (GND), U1.30 (GND), U1.31 (GND), U1.32 (GND), U1.33 (GND), U1.34 (GND), U1.35 (GND), U1.36 (GND), U1.37 (GND), U1.38 (GND), U1.39 (GND), U1.9 (GND)
