File: Vent/Vent.kicad_sch (KiCad schematic)
At the start: 11 parts, among them J2 B2B-XH-A_LF__SN_, J3 Conn_01x03_Pin, SW1 SW_Push, U1 ESP32-H2-MINI-1-H2

Commit message: NOTHING ON THE GROUND PLANE I GUESS BRO
Original-author: Zachariah K. Sharma <zachariah.sharma@gmail.com>
Source-commit: c6036d15c09e4c844a1b63c6872ed82ca575526d
Parts:
- SW1: footprint Button_Switch_THT:SW_PUSH_6mm_H4.3mm -> Button_Switch_SMD:SW_SPST_PTS810
Changed lines of the file:
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@@
 			)
 		)
-		(property "Footprint" "Button_Switch_THT:SW_PUSH_6mm_H4.3mm"
+		(property "Footprint" "Button_Switch_SMD:SW_SPST_PTS810"
 			(at 218.44 143.51 0)
 			(hide yes)
