File: Vent/Vent.kicad_pcb (KiCad board)
At the start: 2 copper layers, 55 x 16 mm, 13 parts, among them J1 SG90_SERVO, J2 AUTO_PROG_TESTPADS, J3 SERVO_5V_BOOST_MODULE, J4 BMS_SPRING_CONTACTS, U1 ESP32-H2-MINI-1-H4S, U2 TPS63031DSK

Commit message: Vent: route SERVO_PWM via west of GND wall, 0 routing-electrical DRC
Previous Plan G connected SERVO_PWM but its F.Cu south leg at x=47 crossed
BB_SW1 diagonal/horizontal and was too close to BMS_SYS_CONTACT diagonal,
yielding 4 routing violations.

New topology: via-on-pad at U1.24 -> B.Cu east-south to (46.7, 15) (stays
west of GND B.Cu vertical wall at x=47.344) -> south to (46.7, 19.8) ->
via to F.Cu in clean band between BB_SW1 horizontal (y=19.31) and J1.3
pad north edge -> short F.Cu hop east at y=19.8 -> enter J1.3 PTH from
north. Shortened upstream B.Cu horizontal endpoint to (46.7, 15) to
eliminate the dangling stub at the old (47, 15) endpoint.

Final DRC: 0 unconnected, 0 clearance/crossing/short, 10 remaining items
are silkscreen-edge/overlap warnings.

Original-author: Zachariah K. Sharma <zachariah.sharma@gmail.com>
Source-commit: 138301c29dd38b6c0487136af83335aa45bf8c60
Routing:
- net SERVO_PWM: track 0.00 -> 34.2 mm, vias 0 -> 2
Changed lines of the file:
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@@
+	)
+	(segment
+		(start 48.5 19.8)
+		(end 48.5 20.58)
+		(width 0.2)
+		(layer "F.Cu")
+		(net 4)
+	)
+	(segment
+		(start 46.7 19.8)
+		(end 48.5 19.8)
+		(width 0.2)
+		(layer "F.Cu")
+		(net 4)
+	)
+	(via
+		(at 22.15 12.75)
+		(size 0.5)
+		(drill 0.3)
+		(layers "F.Cu" "B.Cu")
+		(net 4)
+	)
+	(via
+		(at 46.7 19.8)
+		(size 0.5)
+		(drill 0.3)
+		(layers "F.Cu" "B.Cu")
+		(net 4)
+	)
+	(segment
+		(start 32 15)
+		(end 46.7 15)
+		(width 0.2)
+		(layer "B.Cu")
+		(net 4)
+	)
+	(segment
+		(start 32 12.75)
+		(end 32 15)
+		(width 0.2)
+		(layer "B.Cu")
+		(net 4)
+	)
+	(segment
+		(start 22.15 12.75)
+		(end 32 12.75)
+		(width 0.2)
+		(layer "B.Cu")
+		(net 4)
+	)
+	(segment
+		(start 46.7 15)
+		(end 46.7 19.8)
+		(width 0.2)
+		(layer "B.Cu")
+		(net 4)
 	)
 	(segment
