File: Vent/Vent.kicad_pcb (KiCad board)
At the start: 4 copper layers, 38.1 x 17.6 mm, 26 parts, among them J2 B2B-XH-A_LF__SN_, J3 Conn_01x03_Pin, J4 Conn_01x04_Socket, SW1 SW_Push, U1 ESP32-H2-MINI-1-H2, U4 MCP1640x-xMC

Commit message: idr
Original-author: Zachariah K. Sharma <zachariah.sharma@gmail.com>
Source-commit: 4a91de0f765cb557ab190c59457f2847e7129f6a
Connections:
- U1 pad 49: (no net) -> GND
Routing:
- net GND: track 42.6 -> 63.4 mm, vias 22 -> 33
- net /IO1: track 1.69 -> 11.7 mm, vias 0 -> 2
Changed lines of the file:
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@@
 			(size 0.8 0.8)
 			(layers "F.Cu" "F.Mask" "F.Paste")
+			(net "GND")
 			(zone_connect 2)
 			(thermal_bridge_angle 45)
@@
 			(size 1.45 1.45)
 			(layers "F.Cu" "F.Mask" "F.Paste")
+			(net "GND")
 			(zone_connect 2)
 		)
@@
 			(size 1.45 1.45)
 			(layers "F.Cu" "F.Mask" "F.Paste")
+			(net "GND")
 			(zone_connect 2)
 		)
@@
 			(size 1.45 1.45)
 			(layers "F.Cu" "F.Mask" "F.Paste")
+			(net "GND")
 			(zone_connect 2)
 		)
@@
 			(size 1.45 1.45)
 			(layers "F.Cu" "F.Mask" "F.Paste")
+			(net "GND")
 			(zone_connect 2)
 		)
@@
 			(size 1.45 1.45)
 			(layers "F.Cu" "F.Mask" "F.Paste")
+			(net "GND")
 			(zone_connect 2)
 		)
@@
 			(size 1.45 1.45)
 			(layers "F.Cu" "F.Mask" "F.Paste")
+			(net "GND")
 			(zone_connect 2)
 		)
@@
 			(size 1.45 1.45)
 			(layers "F.Cu" "F.Mask" "F.Paste")
+			(net "GND")
 			(zone_connect 2)
 		)
@@
 			(size 1.45 1.45)
 			(layers "F.Cu" "F.Mask" "F.Paste")
+			(net "GND")
 			(zone_connect 2)
 		)
@@
 	)
 	(segment
+		(start 128.625 73.575)
+		(end 128.625 69.625)
+		(width 0.9)
+		(layer "F.Cu")
+		(net "GND")
+	)
+	(segment
 		(start 139 73.16)
 		(end 138.66 73.16)
@@
 	)
 	(segment
+		(start 136.5 67.6)
+		(end 136.5 66.75)
+		(width 0.7)
+		(layer "F.Cu")
+		(net "GND")
+	)
+	(segment
 		(start 155.675 69.725)
 		(end 155.675 71.475)
 		(width 0.8)
+		(layer "F.Cu")
+		(net "GND")
+	)
+	(segment
+		(start 132.575 73.575)
+		(end 132.575 69.625)
+		(width 0.9)
 		(layer "F.Cu")
 		(net "GND")
@@
 	)
 	(segment
+		(start 136.5 66.75)
+		(end 136.5 66.7)
+		(width 0.7)
+		(layer "F.Cu")
+		(net "GND")
+	)
+	(segment
 		(start 150.356383 67.9275)
 		(end 151.0375 67.9275)
@@
 	)
 	(segment
+		(start 132.575 69.625)
+		(end 128.625 69.625)
+		(width 0.9)
+		(layer "F.Cu")
+		(net "GND")
+	)
+	(segment
 		(start 150.075001 68.208883)
 		(end 150.356383 67.9275)
@@
 	)
 	(segment
+		(start 128.625 71.6)
+		(end 132.575 71.6)
+		(width 0.9)
+		(layer "F.Cu")
+		(net "GND")
+	)
+	(segment
+		(start 128.625 73.575)
+		(end 132.575 73.575)
+		(width 0.9)
+		(layer "F.Cu")
+		(net "GND")
+	)
+	(segment
 		(start 147.81 71.79)
 		(end 147.2 72.4)
@@
 	)
 	(segment
+		(start 136.5 66.7)
+		(end 136.55 66.65)
+		(width 0.7)
+		(layer "F.Cu")
+		(net "GND")
+	)
+	(segment
 		(start 137.5 61.6)
 		(end 138.2 60.9)
@@
 	)
 	(via
+		(at 130.6 69.625)
+		(size 0.6)
+		(drill 0.3)
+		(layers "F.Cu" "B.Cu")
+		(net "GND")
+	)
+	(via
 		(at 152.85 61.15)
 		(size 0.6)
@@
 		(layers "F.Cu" "B.Cu")
 		(free yes)
+		(net "GND")
+	)
+	(via
+		(at 132.575 71.6)
+		(size 0.6)
+		(drill 0.3)
+		(layers "F.Cu" "B.Cu")
+		(net "GND")
+	)
+	(via
+		(at 132.575 69.625)
+		(size 0.6)
+		(drill 0.3)
+		(layers "F.Cu" "B.Cu")
 		(net "GND")
 	)
@@
 	)
 	(via
+		(at 128.625 73.575)
+		(size 0.6)
+		(drill 0.3)
+		(layers "F.Cu" "B.Cu")
+		(net "GND")
+	)
+	(via
+		(at 130.6 71.6)
+		(size 0.6)
+		(drill 0.3)
+		(layers "F.Cu" "B.Cu")
+		(net "GND")
+	)
+	(via
 		(at 140 73.2)
 		(size 0.6)
@@
 	)
 	(via
+		(at 136.5 67.6)
+		(size 0.6)
+		(drill 0.3)
+		(layers "F.Cu" "B.Cu")
+		(net "GND")
+	)
+	(via
 		(at 137.15 61.6)
 		(size 0.6)
@@
 	)
 	(via
+		(at 128.625 71.6)
+		(size 0.6)
+		(drill 0.3)
+		(layers "F.Cu" "B.Cu")
+		(net "GND")
+	)
+	(via
 		(at 123.1 70.35)
 		(size 0.6)
@@
 	)
 	(via
+		(at 128.625 69.625)
+		(size 0.6)
+		(drill 0.3)
+		(layers "F.Cu" "B.Cu")
+		(net "GND")
+	)
+	(via
 		(at 140 68.55)
 		(size 0.6)
@@
 	)
 	(via
+		(at 130.6 73.575)
+		(size 0.6)
+		(drill 0.3)
+		(layers "F.Cu" "B.Cu")
+		(net "GND")
+	)
+	(via
+		(at 132.575 73.575)
+		(size 0.6)
+		(drill 0.3)
+		(layers "F.Cu" "B.Cu")
+		(net "GND")
+	)
+	(via
 		(at 155.7 61.25)
 		(size 0.6)
@@
 		(layers "F.Cu" "B.Cu")
 		(free yes)
+		(net "GND")
+	)
+	(via
+		(at 136.5 66.75)
+		(size 0.6)
+		(drill 0.3)
+		(layers "F.Cu" "B.Cu")
 		(net "GND")
 	)
@@
 	)
 	(segment
+		(start 140.664997 74.000003)
+		(end 140 74.000003)
+		(width 0.25)
+		(layer "F.Cu")
+		(net "/IO1")
+	)
+	(segment
+		(start 140.9 73.765)
+		(end 140.664997 74.000003)
+		(width 0.25)
+		(layer "F.Cu")
+		(net "/IO1")
+	)
+	(segment
 		(start 140.9 73.765)
 		(end 142.555 73.765)
@@
 		(width 0.25)
 		(layer "F.Cu")
+		(net "/IO1")
+	)
+	(segment
+		(start 135.3 68.35)
+		(end 136.45 68.35)
+		(width 0.25)
+		(layer "F.Cu")
+		(net "/IO1")
+	)
+	(segment
+		(start 136.45 68.35)
+		(end 136.5 68.4)
+		(width 0.25)
+		(layer "F.Cu")
+		(net "/IO1")
+	)
+	(via
+		(at 135.3 68.35)
+		(size 0.6)
+		(drill 0.3)
+		(layers "F.Cu" "B.Cu")
+		(net "/IO1")
+	)
+	(via
+		(at 140 74.000003)
+		(size 0.6)
+		(drill 0.3)
+		(layers "F.Cu" "B.Cu")
+		(net "/IO1")
+	)
+	(segment
+		(start 140 74.000003)
+		(end 139.716119 74.000003)
+		(width 0.25)
+		(layer "B.Cu")
+		(net "/IO1")
+	)
+	(segment
+		(start 135.3 69.583884)
+		(end 135.3 68.35)
+		(width 0.25)
+		(layer "B.Cu")
+		(net "/IO1")
+	)
+	(segment
+		(start 139.716119 74.000003)
+		(end 135.3 69.583884)
+		(width 0.25)
+		(layer "B.Cu")
 		(net "/IO1")
 	)
@@
 	(segment
 		(start 129.4 64.5)
-		(end 129.4 67.95)
+		(end 129.4 67.35)
 		(width 0.25)
 		(layer "B.Cu")
@@
 	)
 	(segment
-		(start 135.45 74)
+		(start 129.4 67.35)
+		(end 136.05 74)
+		(width 0.25)
+		(layer "B.Cu")
+		(net "+3.3V")
+	)
+	(segment
+		(start 136.05 74)
 		(end 137.6 74)
 		(width 0.25)
 		(layer "B.Cu")
-		(net "+3.3V")
-	)
-	(segment
-		(start 129.4 67.95)
-		(end 135.45 74)
-		(width 0.25)
-		(layer "B.Cu")
