File: Vent/Vynte PCB.kicad_pcb (KiCad board)
At the start: 4 copper layers, 38.1 x 17.6 mm, 26 parts, among them J2 B2B-XH-A_LF__SN_, J3 Conn_01x03_Pin, J4 Conn_01x04_Socket, SW1 SW_Push, U1 ESP32-H2-MINI-1-H2, U4 MCP1640x-xMC

Commit message: [vent] fix: Remove unused trace
Original-author: Ishan Karmakar <ishan.karmakar24@gmail.com>
Source-commit: ed956880c8593e27f7c3b6b5ca9334a409a4203b
Routing:
- net GND: track 42.6 -> 38.6 mm
Changed lines of the file:
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@@
-	)
-	(segment
-		(start 123.074 67.176)
-		(end 123.074 70.324)
-		(width 0.25)
-		(layer "B.Cu")
-		(net "GND")
 	)
 	(segment
@@
 		(width 0.25)
 		(layer "B.Cu")
-		(net "GND")
-	)
-	(segment
-		(start 123.7 66.55)
-		(end 123.074 67.176)
-		(width 0.25)
-		(layer "B.Cu")
