File: electronics/Autoprogramming/Autoprogramming.kicad_sch (KiCad schematic)
At the start: 0 parts

Commit message: Autoprogramming, Finish off BMS, Add comps to Vent, and do a bunch of mobile stuff
Original-author: Zachariah K. Sharma <zachariah.sharma@gmail.com>
Source-commit: c8fb455aabb0719517b46fd9304eb5e5fb9f4004
Parts:
- added C1: 100nF, PCM_JLCPCB:C_0805, symbol PCM_JLCPCB-Capacitors:0805,100nF
- added C2: 4.7uF, PCM_JLCPCB:C_0805, symbol PCM_JLCPCB-Capacitors:0805,4.7uF
- added J1: TYPE-C-31-M-12, Footprints:HRO_TYPE-C-31-M-12, symbol TYPE-C-31-M-12:TYPE-C-31-M-12
- added J2: Conn_01x05_Pin, symbol Connector:Conn_01x06_Pin
- added Q1, Q2: S8050 J3Y 200-350, PCM_JLCPCB:Q_SOT-23, symbol PCM_JLCPCB-Transistors:NPN,S8050 J3Y 200-350
- added R3, R4: 5.1kΩ, PCM_JLCPCB:R_0603, symbol PCM_JLCPCB-Resistors:0603,5.1kΩ
- added R5, R6: 10kΩ, PCM_JLCPCB:R_0603, symbol PCM_JLCPCB-Resistors:0603,10kΩ
- added U3: CP2102N-A02-GQFN28R, Footprints:IC_CP2102N-A02-GQFN28R, symbol CP2102N-A02-GQFN28R:CP2102N-A02-GQFN28R
Connections:
- new net: Q1.1 (B), R6.2
- new net: C1.1, C2.1, U3.6 (VDD)
- new net: J1.A5 (CC1), R3.1
- new net: J1.B5 (CC2), R4.2
- new net: Q2.1 (B), R5.2
- new net DTR: R6.1, U3.28 (DTR)
- new net EN: J2.1 (Pin_1), Q1.3 (C)
- new net GND: C1.2, C2.2, J1.A1_B12 (GND), J1.B1_A12 (GND), J1.S1 (SHIELD), J1.S2 (SHIELD), J1.S3 (SHIELD), J1.S4 (SHIELD), J2.6 (Pin_6), Q1.2 (E), Q2.2 (E), R3.2, R4.1, U3.29 (EXP), U3.3 (GND)
- new net IO0: J2.2 (Pin_2), Q2.3 (C)
- new net RTS: R5.1, U3.24 (RTS)
- new net RXD0: U3.26 (TXD)
- new net TXD0: U3.25 (RXD)
- new net USB_D+: J1.A6 (DP1), J1.B6 (DP2), J2.3 (Pin_3), U3.4 (D+)
- new net USB_D-: J1.A7 (DN1), J1.B7 (DN2), J2.4 (Pin_4), U3.5 (D-)
- new net VBUS: J1.A4_B9 (VBUS), J1.B4_A9 (VBUS), J2.5 (Pin_5), U3.7 (VREGIN), U3.8 (VBUS)
- no-connect marks 0 -> 19
Other:
- note added: "Autoprogramming Circuit"
- note added: "Connector Pins"
- note added: "USB-to-UART"
