File: electronics/Puck/Vent.kicad_pcb (KiCad board)
At the start: 2 copper layers, 21 parts, among them J1 TYPE-C-31-M-12, Q1 S8050 J3Y 200-350, Q2 S8050 J3Y 200-350, U1 ESP32-S3-WROOM-1, U2 MCP9808T-E_MS, U3 CP2102N-A02-GQFN28R, U4 AP2112K-3.3TRG1

Commit message: Autoprogramming, Finish off BMS, Add comps to Vent, and do a bunch of mobile stuff
Original-author: Zachariah K. Sharma <zachariah.sharma@gmail.com>
Source-commit: c8fb455aabb0719517b46fd9304eb5e5fb9f4004
Parts:
- removed C1: 100nF, PCM_JLCPCB:C_0805
- removed C2: 4.7uF, PCM_JLCPCB:C_0805
- removed Q1, Q2: S8050 J3Y 200-350, PCM_JLCPCB:Q_SOT-23
- removed R5, R6: 10kΩ, PCM_JLCPCB:R_0603
- removed U3: CP2102N-A02-GQFN28R, Footprints:IC_CP2102N-A02-GQFN28R
- added J2: Conn_01x05_Socket, Connector_JST:JST_EH_B6B-EH-A_1x06_P2.50mm_Vertical, F.Cu at (127.4, 100.4)
- R1, R2, U2: moved to B.Cu
- moved U2 33.2 mm to (144.5, 122.0), turned to 180 degrees
- moved R2 22.6 mm to (149.5, 121.8)
- moved R1 21.8 mm to (149.5, 120.8), turned to 0 degrees
- moved J1 19.9 mm to (158.5, 96.5), turned to 90 degrees
- moved C3 7.90 mm to (143.3, 93.8)
- moved C4 7.90 mm to (143.3, 96.0)
- moved C5 7.90 mm to (143.3, 98.2)
- moved R3 7.90 mm to (138.6, 92.2)
- moved R4 7.90 mm to (138.6, 94.5)
- moved R7 7.90 mm to (147.1, 98.2)
- moved R8 7.90 mm to (147.1, 100.5)
- moved C6 3.64 mm to (144.2, 90.2)
- moved U1 0.51 mm to (143.2, 73.7)
Connections:
- J1 pad A6: USB_D+ -> unconnected-(J1-DP1-PadA6)
- J1 pad A7: USB_D- -> unconnected-(J1-DN1-PadA7)
- J1 pad B6: USB_D+ -> unconnected-(J1-DP2-PadB6)
- J1 pad B7: USB_D- -> unconnected-(J1-DN2-PadB7)
Routing:
- net +3.3V: track 0.00 -> 27.4 mm, vias 0 -> 1
- net GND: track 0.00 -> 17.6 mm, vias 0 -> 1
- net IO13: track 0.00 -> 2.41 mm
- net IO11: track 0.00 -> 2.33 mm
- added copper zone on B.Cu, net GND
- added copper zone on F.Cu, net GND
Other:
- board outline added: 36 x 56.8 mm
