File: electronics/Puck/Vent.kicad_sch (KiCad schematic)
At the start: 21 parts, among them J1 TYPE-C-31-M-12, Q1 S8050 J3Y 200-350, Q2 S8050 J3Y 200-350, U1 ESP32-S3-WROOM-1, U2 MCP9808T-E_MS, U3 CP2102N-A02-GQFN28R, U4 AP2112K-3.3TRG1

Commit message: Autoprogramming, Finish off BMS, Add comps to Vent, and do a bunch of mobile stuff
Original-author: Zachariah K. Sharma <zachariah.sharma@gmail.com>
Source-commit: c8fb455aabb0719517b46fd9304eb5e5fb9f4004
Parts:
- removed C1: 100nF, PCM_JLCPCB:C_0805, symbol PCM_JLCPCB-Capacitors:0805,100nF
- removed C2: 4.7uF, PCM_JLCPCB:C_0805, symbol PCM_JLCPCB-Capacitors:0805,4.7uF
- removed Q1, Q2: S8050 J3Y 200-350, PCM_JLCPCB:Q_SOT-23, symbol PCM_JLCPCB-Transistors:NPN,S8050 J3Y 200-350
- removed R5, R6: 10kΩ, PCM_JLCPCB:R_0603, symbol PCM_JLCPCB-Resistors:0603,10kΩ
- removed U3: CP2102N-A02-GQFN28R, Footprints:IC_CP2102N-A02-GQFN28R, symbol CP2102N-A02-GQFN28R:CP2102N-A02-GQFN28R
- added J2: Conn_01x05_Socket, Connector_JST:JST_EH_B6B-EH-A_1x06_P2.50mm_Vertical, symbol Connector:Conn_01x06_Socket
Connections:
- net EN: now also J2.1 (Pin_1)
- net GND: now also J2.6 (Pin_6)
- net IO0: now also J2.2 (Pin_2)
- net USB_D+: now also J2.3 (Pin_3); no longer J1.A6 (DP1), J1.B6 (DP2)
- net USB_D-: now also J2.4 (Pin_4); no longer J1.A7 (DN1), J1.B7 (DN2)
- net VBUS: now also J2.5 (Pin_5)
- no-connect marks 49 -> 36
Other:
- note added: "Connector Sockets"
- note added: "USB"
- note removed: "Autoprogramming Circuit"
- note removed: "PSRAM"
- note removed: "USB-to-UART"
- moved on the sheet: C3, C4, C5, C6, R1, R2, R7, R8, U1, U2, U4
