File: Autoprogramming/Autoprogramming.kicad_sch (KiCad schematic)
At the start: 11 parts, among them J1 TYPE-C-31-M-12, J2 Conn_01x05_Pin, Q1 S8050 J3Y 200-350, Q2 S8050 J3Y 200-350, U3 CP2102N-A02-GQFN28R

Commit message: electronics: Sync latest designs from working directory
- Rename Puck board files (was Vent.kicad_* → Puck.kicad_*)
- Add full Comps libraries (footprints, models, symbols) for all four boards
- Add manufacturing-current/ Gerber outputs and renders for all boards
- Add new components: ESP32-C6-MINI-1 (Puck), ESP32-H2-MINI-1 (Vent), NCU15XH103F60RC (BMS)
- Add PCM JLCPCB passive symbol libraries across all boards
- Add per-project .gitignore files and Autoprogramming/AUTOPROGRAMMING_REVIEW.md
- Add root-level BOM files, sourcing audit, and manufacturing readiness ledger
- Update KiCad design files and Gerbers for BMS, Autoprogramming, and Vent

Co-Authored-By: Claude Sonnet 4.6 <noreply@anthropic.com>

Original-author: Zachariah K. Sharma <zachariah.sharma@gmail.com>
Source-commit: 261c676a3a26a8c60302274465dd756769088335
Parts:
- added U4, U5, U6: TPD2E2U06DCKR, Footprints:SOT65P210X110-3N, symbol TPD2E2U06DCKR:TPD2E2U06DCKR
- C1: footprint PCM_JLCPCB:C_0805 -> PCM_JLCPCB:C_0805_100nF
- C2: footprint PCM_JLCPCB:C_0805 -> PCM_JLCPCB:C_0805_4u7
- J2: value Conn_01x05_Pin -> Conn_01x06_Pin; footprint (none) -> Footprints:JST_EH_B6B-EH-A_1x06_P2.50mm_Vertical
Connections:
- net EN: now also J2.5 (Pin_5), U6.1 (IO1); no longer J2.1 (Pin_1)
- net GND: now also J2.2 (Pin_2), U4.3 (GND), U5.3 (GND), U6.3 (GND); no longer J2.6 (Pin_6)
- net IO0: now also J2.6 (Pin_6), U6.2 (IO2); no longer J2.2 (Pin_2)
- net RXD0: now also J2.3 (Pin_3), U5.1 (IO1)
- net TXD0: now also J2.4 (Pin_4), U5.2 (IO2)
- net USB_D+: now also U4.1 (IO1); no longer J2.3 (Pin_3)
- net USB_D-: now also U4.2 (IO2); no longer J2.4 (Pin_4)
- net VBUS: no longer J2.5 (Pin_5)
- no-connect marks 19 -> 20
Other:
- note added: "+3V3_SENSE"
- note added: "ESD / TVS Protection"
- note added: "Reset / boot TVS"
- note added: "UART TVS"
- note added: "USB data TVS"
