File: BMS/BMS.kicad_pcb (KiCad board)
At the start: 2 copper layers, 23.5 x 72.1 mm, 23 parts, among them J1 USB4105-GF-A, J2 S70-125161545R, J3 S70-125161545R, J4 S70-125161545R, J5 S70-125161545R, J6 Conn_01x01, J7 Conn_01x01, U1 BQ29700DSER, U2 BQ25180YBGR, U3 CSD16406Q3, U4 TPD2E2U06DCKR, U5 CSD16406Q3

Commit message: electronics: Sync latest designs from working directory
- Rename Puck board files (was Vent.kicad_* → Puck.kicad_*)
- Add full Comps libraries (footprints, models, symbols) for all four boards
- Add manufacturing-current/ Gerber outputs and renders for all boards
- Add new components: ESP32-C6-MINI-1 (Puck), ESP32-H2-MINI-1 (Vent), NCU15XH103F60RC (BMS)
- Add PCM JLCPCB passive symbol libraries across all boards
- Add per-project .gitignore files and Autoprogramming/AUTOPROGRAMMING_REVIEW.md
- Add root-level BOM files, sourcing audit, and manufacturing readiness ledger
- Update KiCad design files and Gerbers for BMS, Autoprogramming, and Vent

Co-Authored-By: Claude Sonnet 4.6 <noreply@anthropic.com>

Original-author: Zachariah K. Sharma <zachariah.sharma@gmail.com>
Source-commit: 261c676a3a26a8c60302274465dd756769088335
Parts:
- RT1: value NCP15XH103F03RC -> NCU15XH103F60RC
Routing:
- net GND: track 6.87 -> 20.1 mm
Changed lines of the file:
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@@
 			(net 1 "CELL-")
 			(pintype "passive")
-			(solder_mask_margin 0.102)
+			(solder_mask_margin 0.038)
 			(teardrops
 				(best_length_ratio 0.5)
@@
 			(net 1 "CELL-")
 			(pintype "passive")
-			(solder_mask_margin 0.102)
+			(solder_mask_margin 0.038)
 			(teardrops
 				(best_length_ratio 0.5)
@@
 			(net 1 "CELL-")
 			(pintype "passive")
-			(solder_mask_margin 0.102)
+			(solder_mask_margin 0.038)
 			(teardrops
 				(best_length_ratio 0.5)
@@
 			(net 19 "DOUT")
 			(pintype "passive")
-			(solder_mask_margin 0.102)
+			(solder_mask_margin 0.038)
 			(teardrops
 				(best_length_ratio 0.5)
@@
 		)
 		(embedded_fonts no)
-		(model "${KICAD8_3RD_PARTY}/3dmodels/com_github_CDFER_JLCPCB-Kicad-Library/JLCPCB.3dshapes/C_0402.step"
+		(model "${KICAD9_3DMODEL_DIR}/Capacitor_SMD.3dshapes/C_0402_1005Metric.step"
 			(offset
 				(xyz 0 0 0)
@@
 			(effects
 				(font
-					(size 0.64 0.64)
+					(size 0.8 0.8)
 					(thickness 0.15)
 				)
@@
 			(pinfunction "IO1")
 			(pintype "bidirectional")
-			(solder_mask_margin 0.102)
+			(solder_mask_margin 0.038)
 			(teardrops
 				(best_length_ratio 0.5)
@@
 			(pinfunction "IO2")
 			(pintype "bidirectional")
-			(solder_mask_margin 0.102)
+			(solder_mask_margin 0.038)
 			(teardrops
 				(best_length_ratio 0.5)
@@
 			(pinfunction "GND")
 			(pintype "power_in")
-			(solder_mask_margin 0.102)
+			(solder_mask_margin 0.038)
 			(teardrops
 				(best_length_ratio 0.5)
@@
 		)
 		(embedded_fonts no)
-		(model "${KICAD8_3RD_PARTY}/3dmodels/com_github_CDFER_JLCPCB-Kicad-Library/JLCPCB.3dshapes/C_0603.step"
+		(model "${KICAD9_3DMODEL_DIR}/Capacitor_SMD.3dshapes/C_0603_1608Metric.step"
 			(offset
 				(xyz 0 0 0)
@@
 			(effects
 				(font
-					(size 0.64 0.64)
+					(size 0.8 0.8)
 					(thickness 0.15)
 				)
@@
 			(pinfunction "NC")
 			(pintype "no_connect")
-			(solder_mask_margin 0.102)
+			(solder_mask_margin 0.038)
 			(teardrops
 				(best_length_ratio 0.5)
@@
 			(pinfunction "COUT")
 			(pintype "output")
-			(solder_mask_margin 0.102)
+			(solder_mask_margin 0.038)
 			(teardrops
 				(best_length_ratio 0.5)
@@
 			(pinfunction "DOUT")
 			(pintype "output")
-			(solder_mask_margin 0.102)
+			(solder_mask_margin 0.038)
 			(teardrops
 				(best_length_ratio 0.5)
@@
 			(pinfunction "VSS")
 			(pintype "power_in")
-			(solder_mask_margin 0.102)
+			(solder_mask_margin 0.038)
 			(teardrops
 				(best_length_ratio 0.5)
@@
 			(pinfunction "BAT")
 			(pintype "power_in")
-			(solder_mask_margin 0.102)
+			(solder_mask_margin 0.038)
 			(teardrops
 				(best_length_ratio 0.5)
@@
 			(pinfunction "V-")
 			(pintype "bidirectional")
-			(solder_mask_margin 0.102)
+			(solder_mask_margin 0.038)
 			(teardrops
 				(best_length_ratio 0.5)
@@
 			(net 3 "GND")
 			(pintype "passive")
-			(solder_mask_margin 0.102)
+			(solder_mask_margin 0.038)
 			(teardrops
 				(best_length_ratio 0.5)
@@
 			(net 3 "GND")
 			(pintype "passive")
-			(solder_mask_margin 0.102)
+			(solder_mask_margin 0.038)
 			(teardrops
 				(best_length_ratio 0.5)
@@
 			(net 3 "GND")
 			(pintype "passive")
-			(solder_mask_margin 0.102)
+			(solder_mask_margin 0.038)
 			(thermal_gap 0)
 			(teardrops
@@
 			(net 20 "COUT")
 			(pintype "passive")
-			(solder_mask_margin 0.102)
+			(solder_mask_margin 0.038)
 			(teardrops
 				(best_length_ratio 0.5)
@@
 		)
 		(embedded_fonts no)
-		(model "${KICAD8_3RD_PARTY}/3dmodels/com_github_CDFER_JLCPCB-Kicad-Library/JLCPCB.3dshapes/R_0402.step"
+		(model "${KICAD9_3DMODEL_DIR}/Resistor_SMD.3dshapes/R_0402_1005Metric.step"
 			(offset
 				(xyz 0 0 0)
@@
 		)
 		(embedded_fonts no)
-		(model "${KICAD8_3RD_PARTY}/3dmodels/com_github_CDFER_JLCPCB-Kicad-Library/JLCPCB.3dshapes/R_0402.step"
+		(model "${KICAD9_3DMODEL_DIR}/Resistor_SMD.3dshapes/R_0402_1005Metric.step"
 			(offset
 				(xyz 0 0 0)
@@
 		)
 		(embedded_fonts no)
-		(model "${KICAD8_3RD_PARTY}/3dmodels/com_github_CDFER_JLCPCB-Kicad-Library/JLCPCB.3dshapes/R_0402.step"
+		(model "${KICAD9_3DMODEL_DIR}/Resistor_SMD.3dshapes/R_0402_1005Metric.step"
 			(offset
 				(xyz 0 0 0)
@@
 		)
 		(fp_line
-			(start 4.47 2.6)
-			(end 4.47 1.32)
-			(stroke
-				(width 0.2)
-				(type solid)
-			)
-			(layer "F.SilkS")
-		)
-		(fp_line
-			(start 4.47 -2.65)
-			(end 4.47 -1.4)
-			(stroke
-				(width 0.2)
-				(type solid)
-			)
-			(layer "F.SilkS")
-		)
-		(fp_line
-			(start -4.47 1.32)
-			(end -4.47 2.6)
-			(stroke
-				(width 0.2)
-				(type solid)
-			)
-			(layer "F.SilkS")
-		)
-		(fp_line
-			(start -4.47 -2.65)
-			(end -4.47 -1.4)
-			(stroke
-				(width 0.2)
-				(type solid)
-			)
-			(layer "F.SilkS")
-		)
-		(fp_circle
-			(center -3.25 -6)
-			(end -3.15 -6)
-			(stroke
-				(width 0.2)
-				(type solid)
-			)
-			(fill no)
-			(layer "F.SilkS")
-		)
-		(fp_line
 			(start 5.07 2.85)
 			(end 5.07 -5.58)
@@
 			(pinfunction "SHELL_GND")
 			(pintype "power_in")
-			(solder_mask_margin 0.102)
+			(solder_mask_margin 0.038)
 			(teardrops
 				(best_length_ratio 0.5)
@@
 			(pinfunction "SHELL_GND")
 			(pintype "power_in")
-			(solder_mask_margin 0.102)
+			(solder_mask_margin 0.038)
 			(teardrops
 				(best_length_ratio 0.5)
@@
 			(pinfunction "SHELL_GND")
 			(pintype "power_in")
-			(solder_mask_margin 0.102)
+			(solder_mask_margin 0.038)
 			(teardrops
 				(best_length_ratio 0.5)
@@
 			(pinfunction "SHELL_GND")
 			(pintype "power_in")
-			(solder_mask_margin 0.102)
+			(solder_mask_margin 0.038)
 			(teardrops
 				(best_length_ratio 0.5)
@@
 		)
 		(embedded_fonts no)
-		(model "${KICAD8_3RD_PARTY}/3dmodels/com_github_CDFER_JLCPCB-Kicad-Library/JLCPCB.3dshapes/R_0402.step"
+		(model "${KICAD9_3DMODEL_DIR}/Resistor_SMD.3dshapes/R_0402_1005Metric.step"
 			(offset
 				(xyz 0 0 0)
@@
 		)
 		(embedded_fonts no)
-		(model "${KICAD8_3RD_PARTY}/3dmodels/com_github_CDFER_JLCPCB-Kicad-Library/JLCPCB.3dshapes/C_0402.step"
+		(model "${KICAD9_3DMODEL_DIR}/Capacitor_SMD.3dshapes/C_0402_1005Metric.step"
 			(offset
 				(xyz 0 0 0)
@@
 		)
 		(embedded_fonts no)
-		(model "${KICAD8_3RD_PARTY}/3dmodels/com_github_CDFER_JLCPCB-Kicad-Library/JLCPCB.3dshapes/C_0402.step"
+		(model "${KICAD9_3DMODEL_DIR}/Capacitor_SMD.3dshapes/C_0402_1005Metric.step"
 			(offset
 				(xyz 0 0 0)
@@
 			(effects
 				(font
-					(size 0.393701 0.393701)
-					(thickness 0.098425)
+					(size 0.8 0.8)
+					(thickness 0.15)
 				)
 			)
 		)
-		(property "Value" "NCP15XH103F03RC"
+		(property "Value" "NCU15XH103F60RC"
 			(at 2.3 0.88 0)
 			(layer "F.Fab")
@@
 			)
 		)
-		(property "SnapEDA_Link" "https://www.snapeda.com/parts/NCP15XH103F03RC/Murata/view-part/?ref=snap"
+		(property "SnapEDA_Link" "https://www.digikey.com/en/products/detail/murata-electronics/NCU15XH103F60RC/9686714"
 			(at 0 0 0)
 			(unlocked yes)
@@
 			)
 		)
-		(property "MP" "NCP15XH103F03RC"
+		(property "MP" "NCU15XH103F60RC"
 			(at 0 0 0)
 			(unlocked yes)
@@
 			)
 		)
-		(property "Check_prices" "https://www.snapeda.com/parts/NCP15XH103F03RC/Murata/view-part/?ref=eda"
+		(property "Check_prices" "https://www.digikey.com/en/products/detail/murata-electronics/NCU15XH103F60RC/9686714"
 			(at 0 0 0)
 			(unlocked yes)
@@
 			(net 18 "Net-(U2-TS{slash}MR)")
 			(pintype "passive")
-			(solder_mask_margin 0.102)
+			(solder_mask_margin 0.038)
 			(teardrops
 				(best_length_ratio 0.5)
@@
 			(net 3 "GND")
 			(pintype "passive")
-			(solder_mask_margin 0.102)
+			(solder_mask_margin 0.038)
 			(teardrops
 				(best_length_ratio 0.5)
@@
 		)
 		(embedded_fonts no)
-		(model "${KIPRJMOD}/Comps/Models/NCP15XH103F03RC.step"
+		(model "${KIPRJMOD}/Comps/Models/NCU15XH103F60RC.step"
 			(offset
 				(xyz 0 0 0)
@@
 		)
 		(embedded_fonts no)
-		(model "${KICAD8_3RD_PARTY}/3dmodels/com_github_CDFER_JLCPCB-Kicad-Library/JLCPCB.3dshapes/R_0402.step"
+		(model "${KICAD9_3DMODEL_DIR}/Resistor_SMD.3dshapes/R_0402_1005Metric.step"
 			(offset
 				(xyz 0 0 0)
@@
 		)
 		(embedded_fonts no)
-		(model "${KICAD8_3RD_PARTY}/3dmodels/com_github_CDFER_JLCPCB-Kicad-Library/JLCPCB.3dshapes/R_0402.step"
+		(model "${KICAD9_3DMODEL_DIR}/Resistor_SMD.3dshapes/R_0402_1005Metric.step"
 			(offset
 				(xyz 0 0 0)
@@
 			(unlocked yes)
 			(layer "B.SilkS")
+			(hide yes)
 			(effects
 				(font
@@
 			(unlocked yes)
 			(layer "B.SilkS")
+			(hide yes)
 			(effects
 				(font
@@
 			(unlocked yes)
 			(layer "B.SilkS")
+			(hide yes)
 			(effects
 				(font
@@
 			(unlocked yes)
 			(layer "B.SilkS")
+			(hide yes)
 			(effects
 				(font
@@
 	)
 	(segment
+		(start 85.68 40)
+		(end 85.68 44.18)
+		(width 0.5)
+		(layer "F.Cu")
+		(net 3)
+	)
+	(segment
+		(start 89 80.5)
+		(end 87 79.28)
+		(width 0.25)
+		(layer "F.Cu")
+		(net 3)
+	)
+	(segment
+		(start 86.8 44.755)
+		(end 85.68 44.18)
+		(width 0.25)
+		(layer "F.Cu")
+		(net 3)
+	)
+	(segment
 		(start 89.1 76.5)
 		(end 89.1 76.1)
@@
 	)
 	(segment
+		(start 93.2 44.755)
+		(end 94.32 44.18)
+		(width 0.25)
+		(layer "F.Cu")
+		(net 3)
+	)
+	(segment
 		(start 89.1 76.1)
 		(end 88.5 75.5)
@@
 	)
 	(segment
+		(start 94.32 40)
+		(end 94.32 44.18)
+		(width 0.5)
+		(layer "F.Cu")
+		(net 3)
+	)
+	(segment
 		(start 92.345 91.975)
 		(end 92.345 91)
@@
 		(hatch edge 0.5)
 		(connect_pads
-			(clearance 0.5)
+			(clearance 0.15)
 		)
 		(min_thickness 0.25)
